File: seths 4layer nano.sch (EAGLE design)
At the start: 30 parts, among them IC1 FT232RL, J1 1981568-1, Q1 CSTCR6M00G53Z, X1 TSW-115-07-G-S, X2 TSW-115-07-G-S

Commit message: Add files via upload
updating this since it hasn't been in a while.
Parts:
- U1: device UA78M05CDCYR:UA78M05CDCYR -> UA78M05CDCYR:UA78M05CDCYRDCY4-L
Connections:
- net GND: now also IC1.TEST
Changed lines of the file:
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@@
 <part name="J1" library="1981568-1" deviceset="1981568-1" device=""/>
 <part name="U$1" library="MBR0520LT1G" deviceset="MBR0520LT1G" device=""/>
-<part name="U1" library="UA78M05CDCYR" deviceset="UA78M05CDCYR" device=""/>
+<part name="U1" library="UA78M05CDCYR" deviceset="UA78M05CDCYR" device="DCY4-L"/>
 <part name="X1" library="con-samtec" library_urn="urn:adsk.eagle:library:184" deviceset="TSW-115-*-G-S" device="" technology="07"/>
 <part name="X2" library="con-samtec" library_urn="urn:adsk.eagle:library:184" deviceset="TSW-115-*-G-S" device="" technology="07"/>
@@
 <junction x="195.58" y="104.14"/>
 <wire x1="195.58" y1="101.6" x2="195.58" y2="104.14" width="0.1524" layer="91"/>
+<pinref part="IC1" gate="G$1" pin="TEST"/>
+<wire x1="198.12" y1="124.46" x2="195.58" y2="124.46" width="0.1524" layer="91"/>
+<wire x1="195.58" y1="124.46" x2="195.58" y2="121.92" width="0.1524" layer="91"/>
+<junction x="195.58" y="121.92"/>
 </segment>
 <segment>
@@
 <pinref part="R2" gate="G$1" pin="2"/>
 <label x="50.8" y="73.66" size="1.778" layer="95"/>
+<wire x1="50.8" y1="86.36" x2="50.8" y2="71.12" width="0.1524" layer="91"/>
+<wire x1="50.8" y1="86.36" x2="7.62" y2="86.36" width="0.1524" layer="91"/>
 <pinref part="U1" gate="A" pin="OUT"/>
-<wire x1="58.42" y1="101.6" x2="58.42" y2="86.36" width="0.1524" layer="91"/>
-<wire x1="58.42" y1="86.36" x2="50.8" y2="86.36" width="0.1524" layer="91"/>
-<wire x1="50.8" y1="86.36" x2="50.8" y2="71.12" width="0.1524" layer="91"/>
+<wire x1="7.62" y1="86.36" x2="7.62" y2="101.6" width="0.1524" layer="91"/>
 </segment>
 <segment>
@@
 <wire x1="25.4" y1="66.04" x2="25.4" y2="71.12" width="0.1524" layer="91"/>
 <label x="25.4" y="71.12" size="1.778" layer="95"/>
+<wire x1="7.62" y1="71.12" x2="25.4" y2="71.12" width="0.1524" layer="91"/>
+<wire x1="7.62" y1="71.12" x2="7.62" y2="78.74" width="0.1524" layer="91"/>
+<wire x1="7.62" y1="78.74" x2="45.72" y2="78.74" width="0.1524" layer="91"/>
+<wire x1="45.72" y1="78.74" x2="45.72" y2="91.44" width="0.1524" layer="91"/>
+<wire x1="45.72" y1="91.44" x2="58.42" y2="91.44" width="0.1524" layer="91"/>
 <pinref part="U1" gate="A" pin="IN"/>
-<wire x1="7.62" y1="101.6" x2="7.62" y2="71.12" width="0.1524" layer="91"/>
-<wire x1="7.62" y1="71.12" x2="25.4" y2="71.12" width="0.1524" layer="91"/>
-</segment>
-<segment>
+<wire x1="58.42" y1="91.44" x2="58.42" y2="101.6" width="0.1524" layer="91"/>
+</segment>
+<segment>

Commit message: updating schematic and BRD files
updating the schematic and board files.
Changed lines of the file:
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@@
 <sheet>
 <plain>
+<wire x1="-17.78" y1="215.9" x2="304.8" y2="215.9" width="0.1524" layer="94"/>
+<wire x1="304.8" y1="215.9" x2="304.8" y2="25.4" width="0.1524" layer="94"/>
+<wire x1="304.8" y1="25.4" x2="-17.78" y2="25.4" width="0.1524" layer="94"/>
+<wire x1="-17.78" y1="25.4" x2="-17.78" y2="215.9" width="0.1524" layer="94"/>
 </plain>
 <instances>
